Commit message: Fix names of pkg

File: urdf/ur5.urdf.xacro (robot description, xacro)
@@ -2,5 +2,5 @@
 <robot xmlns:xacro="http://www.ros.org/wiki/xacro">
   <!--xacro:include filename="$(find ur5_vacuum)/urdf/ur.transmission.xacro" /-->
-  <xacro:include filename="$(find ur5_vacuum)/urdf/common.gazebo.xacro" />
+  <xacro:include filename="$(find subbotinny_ur5_vacuum)/urdf/common.gazebo.xacro" />
   <!-- Inertia parameters -->
   <xacro:property name="base_mass" value="4.0" />  <!-- This mass might be incorrect -->

File: urdf/ur5_joint_limited_robot.urdf.xacro (robot description, xacro)
@@ -4,12 +4,12 @@
   <!-- common stuff -->
   <!-- <xacro:include filename="$(find ur5_vacuum)/urdf/common.gazebo.xacro" /> -->
-  <xacro:include filename="$(find ur5_vacuum)/urdf/ur5.material.xacro" />
+  <xacro:include filename="$(find subbotinny_ur5_vacuum)/urdf/ur5.material.xacro" />
   <!-- ur5 -->
-  <xacro:include filename="$(find ur5_vacuum)/urdf/ur5.urdf.xacro" />
+  <xacro:include filename="$(find subbotinny_ur5_vacuum)/urdf/ur5.urdf.xacro" />
   <xacro:macro name="box" params="suffix x y">
     <link name="box_${suffix}">
       <visual>
         <geometry>
-          <mesh scale = "0.005 0.005 0.005" filename="package://ur5_vacuum/meshes/box.stl"/>
+          <mesh scale = "0.005 0.005 0.005" filename="package://subbotinny_ur5_vacuum/meshes/box.stl"/>
         </geometry>
         <xacro:insert_block name="pink" />
@@ -17,5 +17,5 @@
       <collision>
         <geometry>
-          <mesh scale = "0.005 0.005 0.005" filename="package://ur5_vacuum/meshes/box.stl"/>
+          <mesh scale = "0.005 0.005 0.005" filename="package://subbotinny_ur5_vacuum/meshes/box.stl"/>
         </geometry>
       </collision>
@@ -68,5 +68,5 @@
     <visual>
       <geometry>
-        <mesh scale = "0.0025 0.0025 0.0025" filename="package://ur5_vacuum/meshes/board.stl" />
+        <mesh scale = "0.0025 0.0025 0.0025" filename="package://subbotinny_ur5_vacuum/meshes/board.stl" />
       </geometry>
       <xacro:insert_block name="white" />
@@ -74,5 +74,5 @@
     <collision>
       <geometry>
-        <mesh scale = "0.0025 0.0025 0.0025" filename="package://ur5_vacuum/meshes/board.stl" />
+        <mesh scale = "0.0025 0.0025 0.0025" filename="package://subbotinny_ur5_vacuum/meshes/board.stl" />
       </geometry>
     </collision>
