Commit message: Added: ros_control, camera

File: urdf/common.gazebo.xacro (robot description, xacro)
@@ -2,23 +2,53 @@
 <robot xmlns:xacro="http://ros.org/wiki/xacro">
   <gazebo>
-    <!--plugin name="ros_control" filename="libgazebo_ros_control.so"-->
-      <!--robotNamespace>/</robotNamespace-->
-      <!--robotSimType>gazebo_ros_control/DefaultRobotHWSim</robotSimType-->
-    <!--plugin-->
-    <!-- loading plugin: mimic joints works in gazebo now -->
-<!--
-    <plugin name="gazebo_ros_power_monitor_controller" filename="libgazebo_ros_power_monitor.so">
-      <alwaysOn>true</alwaysOn>
-      <updateRate>1.0</updateRate>
-      <timeout>5</timeout>
-      <powerStateTopic>power_state</powerStateTopic>
-      <powerStateRate>10.0</powerStateRate>
-      <fullChargeCapacity>87.78</fullChargeCapacity>
-      <dischargeRate>-474</dischargeRate>
-      <chargeRate>525</chargeRate>
-      <dischargeVoltage>15.52</dischargeVoltage>
-      <chargeVoltage>16.41</chargeVoltage>
+    <plugin filename="libgazebo_ros_control.so" name="gazebo_ros_control">
+      <robotNamespace>/ur5_sub</robotNamespace>
     </plugin>
--->
+  </gazebo>
+  <gazebo>
+    <plugin name="gazebo_ros_vacuum_gripper" filename="libgazebo_ros_vacuum_gripper.so">
+      <robotNamespace>/ur5_sub</robotNamespace>
+      <bodyName>vacuum_gripper</bodyName>
+      <topicName>grasping</topicName>
+      <maxForce>50</maxForce>
+      <maxDistance>0.05</maxDistance>
+      <minDistance>0.01</minDistance>
+    </plugin>
+  </gazebo>
+  <gazebo reference="camera">
+    <sensor type="camera" name="camera">
+      <update_rate>30.0</update_rate>
+      <camera name="camera">
+        <horizontal_fov>${radians(100)}</horizontal_fov>
+        <image>
+          <width>640</width>
+          <height>480</height>
+          <format>R8G8B8</format>
+        </image>
+        <clip>
+          <near>0.005</near>
+          <far>300</far>
+        </clip>
+        <noise>
+          <type>gaussian</type>
+          <mean>0.0</mean>
+          <stddev>0.005</stddev>
+        </noise>
+      </camera>
+      <plugin name="camera_controller" filename="libgazebo_ros_camera.so">
+        <alwaysOn>true</alwaysOn>
+        <updateRate>0.0</updateRate>
+        <cameraName>camera</cameraName>
+        <imageTopicName>image_raw</imageTopicName>
+        <cameraInfoTopicName>camera_info</cameraInfoTopicName>
+        <frameName>camera</frameName>
+        <hackBaseline>0.07</hackBaseline>
+        <distortionK1>0.0</distortionK1>
+        <distortionK2>0.0</distortionK2>
+        <distortionK3>0.0</distortionK3>
+        <distortionT1>0.0</distortionT1>
+        <distortionT2>0.0</distortionT2>
+      </plugin>
+    </sensor>
   </gazebo>
 </robot>

File: urdf/ur5.urdf.xacro (robot description, xacro)
@@ -1,6 +1,5 @@
 <?xml version="1.0"?>
 <robot xmlns:xacro="http://www.ros.org/wiki/xacro">
-  <!--xacro:include filename="$(find ur5_vacuum)/urdf/ur.transmission.xacro" /-->
-  <xacro:include filename="$(find subbotinny_ur5_vacuum)/urdf/common.gazebo.xacro" />
+  <xacro:include filename="$(find subbotinny_ur5_vacuum)/urdf/ur.transmission.xacro" />
   <!-- Inertia parameters -->
   <xacro:property name="base_mass" value="4.0" />  <!-- This mass might be incorrect -->
@@ -313,4 +312,10 @@
       </material>
     </visual>
+    <collision>
+      <origin rpy="0 0 0" xyz="0 0 0"/>
+      <geometry>
+        <cylinder radius="0.005" length="0.01"/>
+      </geometry>
+    </collision>
     <inertial>
       <origin rpy="0 0 0" xyz="0.000000 0.000000 0.000000"/>
@@ -327,15 +332,5 @@
     <dynamics damping="0.0" friction="10"/>
   </joint>
-  <gazebo>
-    <plugin name="gazebo_ros_vacuum_gripper" filename="libgazebo_ros_vacuum_gripper.so">
-      <robotNamespace>/ur5/vacuum_gripper</robotNamespace>
-      <bodyName>vacuum_gripper</bodyName>
-      <topicName>grasping</topicName>
-  <maxForce>50</maxForce>
-      <maxDistance>0.05</maxDistance>
-      <minDistance>0.01</minDistance>
-    </plugin>
-  </gazebo>
-    <!--xacro:ur_arm_transmission prefix="${prefix}" /-->
+    <xacro:ur_arm_transmission prefix="${prefix}" />
     <!--xacro:ur_arm_gazebo prefix="${prefix}" /-->
     <!-- ROS base_link to UR 'Base' Coordinates transform -->

File: urdf/ur5_joint_limited_robot.urdf.xacro (robot description, xacro)
@@ -7,4 +7,5 @@
   <!-- ur5 -->
   <xacro:include filename="$(find subbotinny_ur5_vacuum)/urdf/ur5.urdf.xacro" />
+  <xacro:include filename="$(find subbotinny_ur5_vacuum)/urdf/common.gazebo.xacro" />
   <xacro:macro name="box" params="suffix x y">
     <link name="box_${suffix}">
@@ -65,4 +66,30 @@
   <xacro:box suffix="2" x="2" y="2" />
   <xacro:box suffix="3" x="3" y="2" />
+  <link name="camera_stand">
+    <visual>
+      <geometry>
+        <cylinder length="0.025" radius="0.1" />
+      </geometry>
+      <origin xyz="0 0 0" />
+      <xacro:insert_block name="pastel_blue" />
+    </visual>
+    <collision>
+      <geometry>
+        <cylinder length="0.025" radius="0.1" />
+      </geometry>
+      <origin xyz="0 0 0" />
+    </collision>
+  </link>
+  <joint name="camera_stand_joint" type="fixed">
+    <parent link="table" />
+    <child link="camera_stand" />
+    <origin xyz="-0.2 0 0.2125" rpy="0 0 0" />
+  </joint>
+  <link name="camera" />
+  <joint name="camera_joint" type="fixed">
+    <parent link="camera_stand" />
+    <child link="camera" />
+    <origin xyz="0 0 0.05" rpy="0 ${radians(-90)} 0" />
+  </joint>
   <link name="PCB">
     <visual>
@@ -81,5 +108,5 @@
     <parent link="table" />
     <child link="PCB" />
-    <origin xyz="-0.1 0.1 0.205" rpy="0.0 0.0 ${pi/2}"/>
+    <origin xyz="-0.1 0.2 0.205" rpy="0.0 0.0 ${pi/2}"/>
   </joint>
 </robot>

Commit message: Added: python script moving to camera

File: urdf/common.gazebo.xacro (robot description, xacro)
@@ -1,4 +1,8 @@
 <?xml version="1.0"?>
 <robot xmlns:xacro="http://ros.org/wiki/xacro">
+  <gazebo reference="table">
+    <minDepth>0.001</minDepth>
+    <material>Gazebo/SkyBlue</material>
+  </gazebo>
   <gazebo>
     <plugin filename="libgazebo_ros_control.so" name="gazebo_ros_control">
@@ -11,7 +15,7 @@
       <bodyName>vacuum_gripper</bodyName>
       <topicName>grasping</topicName>
-      <maxForce>50</maxForce>
-      <maxDistance>0.05</maxDistance>
-      <minDistance>0.01</minDistance>
+      <maxForce>1000</maxForce>
+      <maxDistance>5</maxDistance>
+      <minDistance>0.001</minDistance>
     </plugin>
   </gazebo>
