Commit message: gazebo.launch with sdf world

File: subbotinny_ur5_arm/urdf/ur5_pcb_table.urdf.xacro (robot description, xacro)
@@ -9,24 +9,4 @@
   <xacro:include filename="$(find subbotinny_ur5_vacuum)/urdf/common.gazebo.xacro" />
   <xacro:include filename="$(find subbotinny_ur5_vacuum)/urdf/pcb_components.urdf.xacro" />
-  <xacro:macro name="box" params="suffix x y">
-    <link name="box_${suffix}">
-      <visual>
-        <geometry>
-          <mesh scale = "0.005 0.005 0.005" filename="package://subbotinny_ur5_vacuum/meshes/box.stl"/>
-        </geometry>
-        <xacro:insert_block name="pink" />
-      </visual>
-      <collision>
-        <geometry>
-          <mesh scale = "0.005 0.005 0.005" filename="package://subbotinny_ur5_vacuum/meshes/box.stl"/>
-        </geometry>
-      </collision>
-    </link>
-    <joint name="box_${suffix}_joint" type="fixed">
-      <parent link="table" />
-      <child link="box_${suffix}" />
-      <origin xyz="${x * -0.1} ${y * -0.1} 0.2" />
-    </joint>
-  </xacro:macro>
   <!-- arm -->
   <xacro:ur5_robot prefix="" joint_limited="true"
@@ -39,76 +19,15 @@
   />
   <link name="world" />
-  <link name="table">
-    <visual>
-      <geometry>
-        <box size="1 1 0.2" />
-      </geometry>
-      <origin xyz="0 0 0.1" />
-        <xacro:insert_block name="pastel_blue" />
-    </visual>
-    <collision>
-      <geometry>
-        <box size="1 1 0.2" />
-      </geometry>
-      <origin xyz="0 0 0.1" />
-    </collision>
-  </link>
+  <!-- <xacro:rc0805 prefix="1" box_num="3"/> -->
   <joint name="world_joint" type="fixed">
     <parent link="world" />
-    <child link = "table" />
-    <origin xyz="0 0 0" rpy="0.0 0.0 0.0" />
-  </joint>
-  <joint name="table_joint" type="fixed">
-    <parent link="table" />
     <child link = "base_link" />
-    <origin xyz="0.4 0 0.2" rpy="0.0 0.0 0.0" />
-  </joint> >
-  <xacro:box suffix="1" x="1" y="2" />
-  <xacro:box suffix="2" x="2" y="2" />
-  <xacro:box suffix="3" x="3" y="2" />
-  <!-- <xacro:rc0805 prefix="1" box_num="3"/> -->
-  <link name="camera_stand">
-    <visual>
-      <geometry>
-        <cylinder length="0.025" radius="0.1" />
-      </geometry>
-      <origin xyz="0 0 0" />
-      <xacro:insert_block name="pastel_blue" />
-    </visual>
-    <collision>
-      <geometry>
-        <cylinder length="0.025" radius="0.1" />
-      </geometry>
-      <origin xyz="0 0 0" />
-    </collision>
-  </link>
-  <joint name="camera_stand_joint" type="fixed">
-    <parent link="table" />
-    <child link="camera_stand" />
-    <origin xyz="-0.2 0 0.2125" rpy="0 0 0" />
+    <origin xyz="0 -0.4 0.1" rpy="0.0 0.0 0.0" />
   </joint>
   <link name="camera" />
   <joint name="camera_joint" type="fixed">
-    <parent link="camera_stand" />
+    <parent link="world" />
     <child link="camera" />
-    <origin xyz="0 0 0.05" rpy="0 ${radians(-90)} 0" />
-  </joint>
-  <link name="PCB">
-    <visual>
-      <geometry>
-        <mesh scale = "0.0025 0.0025 0.0025" filename="package://subbotinny_ur5_vacuum/meshes/board.stl" />
-      </geometry>
-      <xacro:insert_block name="white" />
-    </visual>
-    <collision>
-      <geometry>
-        <mesh scale = "0.0025 0.0025 0.0025" filename="package://subbotinny_ur5_vacuum/meshes/board.stl" />
-      </geometry>
-    </collision>
-  </link>
-  <joint name="board_joint" type="fixed">
-    <parent link="table" />
-    <child link="PCB" />
-    <origin xyz="-0.1 0.2 0.205" rpy="0.0 0.0 ${pi/2}"/>
+    <origin xyz="0 0.4 0.11" rpy="0 ${radians(-90)} 0" />
   </joint>
 </robot>

Commit message: Fixed vibration of model

File: subbotinny_ur5_arm/urdf/ur5_pcb_table.urdf.xacro (robot description, xacro)
@@ -23,5 +23,5 @@
     <parent link="world" />
     <child link = "base_link" />
-    <origin xyz="0 -0.4 0.1" rpy="0.0 0.0 0.0" />
+    <origin xyz="0 -0.4 0.105" rpy="0.0 0.0 0.0" />
   </joint>
   <link name="camera" />
