Commit message: Vacuum gripper fix

File: subbotinny_ur5_arm/urdf/common.gazebo.xacro (robot description, xacro)
@@ -12,10 +12,10 @@
   <gazebo>
     <plugin name="gazebo_ros_vacuum_gripper" filename="libgazebo_ros_vacuum_gripper.so">
-      <robotNamespace>/ur5_sub</robotNamespace>
+      <robotNamespace>/ur5_sub/vacuum_gripper</robotNamespace>
       <bodyName>vacuum_gripper</bodyName>
       <topicName>grasping</topicName>
-      <maxForce>1000</maxForce>
-      <maxDistance>5</maxDistance>
-      <minDistance>0.001</minDistance>
+      <maxForce>50</maxForce>
+      <maxDistance>0.05</maxDistance>
+      <minDistance>0.01</minDistance>
     </plugin>
   </gazebo>
@@ -26,10 +26,10 @@
         <horizontal_fov>${radians(100)}</horizontal_fov>
         <image>
-          <width>640</width>
-          <height>480</height>
+          <width>800</width>
+          <height>800</height>
           <format>R8G8B8</format>
         </image>
         <clip>
-          <near>0.005</near>
+          <near>0.02</near>
           <far>300</far>
         </clip>
@@ -47,5 +47,5 @@
         <cameraInfoTopicName>camera_info</cameraInfoTopicName>
         <frameName>camera</frameName>
-        <hackBaseline>0.07</hackBaseline>
+        <hackBaseline>0.0</hackBaseline>
         <distortionK1>0.0</distortionK1>
         <distortionK2>0.0</distortionK2>

File: subbotinny_ur5_arm/urdf/ur5.urdf.xacro (robot description, xacro)
@@ -11,5 +11,4 @@
   <xacro:property name="wrist_3_mass" value="0.1879" />
   <xacro:property name="height3" value="1" /> <!-- Link 3 -->
-  <xacro:property name="camera_link" value="0.02" /> <!-- Size of square 'camera' box -->
   <xacro:property name="axel_offset" value="0.05" /> <!-- Space btw top of beam and the each joint -->
   <xacro:property name="shoulder_cog" value="0.0 0.00193 -0.02561" />
@@ -301,35 +300,29 @@
       </collision>
     </link>
-  <link name="vacuum_gripper">
-    <gravity>0</gravity>
-    <visual>
-      <origin rpy="0 0 0" xyz="0 0 0"/>
-      <geometry>
-        <cylinder radius="0.005" length="0.01"/>
-      </geometry>
-      <material name="transparent">
-        <color rgba="0 0 0 0"/>
-      </material>
-    </visual>
-    <collision>
-      <origin rpy="0 0 0" xyz="0 0 0"/>
-      <geometry>
-        <cylinder radius="0.005" length="0.01"/>
-      </geometry>
-    </collision>
-    <inertial>
-      <origin rpy="0 0 0" xyz="0.000000 0.000000 0.000000"/>
-      <mass value="0.0001"/>
-      <inertia ixx="1e-08" ixy="0" ixz="0" iyy="1e-08" iyz="0" izz="1e-08"/>
-    </inertial>
-  </link>
-  <joint name="gripper_joint" type="fixed">
-    <axis xyz="1 0 0" />
-    <parent link="ee_link" />
-    <child link="vacuum_gripper" />
-    <origin rpy="0 1.5708 0" xyz="0.01 0 0" />
-    <limit effort="50" velocity="50" lower="0" upper="0" />
-    <dynamics damping="0.0" friction="10"/>
-  </joint>
+    <link name="vacuum_gripper">
+      <gravity>0</gravity>
+      <visual>
+        <origin rpy="0 0 0" xyz="0 0 0"/>
+        <geometry>
+          <cylinder radius="0.005" length="0.01"/>
+        </geometry>
+        <material name="transparent">
+          <color rgba="0 0 0 0"/>
+        </material>
+      </visual>
+      <inertial>
+        <origin rpy="0 0 0" xyz="0.000000 0.000000 0.000000"/>
+        <mass value="0.0001"/>
+        <inertia ixx="1e-08" ixy="0" ixz="0" iyy="1e-08" iyz="0" izz="1e-08"/>
+      </inertial>
+    </link>
+    <joint name="gripper_joint" type="fixed">
+      <axis xyz="1 0 0" />
+      <parent link="ee_link" />
+      <child link="vacuum_gripper" />
+      <origin rpy="0 1.5708 0" xyz="0.01 0 0" />
+<!--       <limit effort="50" velocity="50" lower="0" upper="0" />
+      <dynamics damping="0.0" friction="10"/> -->
+    </joint>
     <xacro:ur_arm_transmission prefix="${prefix}" />
     <!--xacro:ur_arm_gazebo prefix="${prefix}" /-->

File: subbotinny_ur5_arm/urdf/ur5_pcb_table.urdf.xacro (robot description, xacro)
@@ -8,5 +8,4 @@
   <xacro:include filename="$(find subbotinny_ur5_vacuum)/urdf/ur5.urdf.xacro" />
   <xacro:include filename="$(find subbotinny_ur5_vacuum)/urdf/common.gazebo.xacro" />
-  <xacro:include filename="$(find subbotinny_ur5_vacuum)/urdf/pcb_components.urdf.xacro" />
   <!-- arm -->
   <xacro:ur5_robot prefix="" joint_limited="true"
@@ -29,5 +28,5 @@
     <parent link="world" />
     <child link="camera" />
-    <origin xyz="0 0.4 0.11" rpy="0 ${radians(-90)} 0" />
+    <origin xyz="0 0.3 0.2" rpy="0 ${radians(-90)} 0" />
   </joint>
 </robot>

Commit message: Camera fix

File: subbotinny_ur5_arm/urdf/common.gazebo.xacro (robot description, xacro)
@@ -1,58 +1,56 @@
 <?xml version="1.0"?>
 <robot xmlns:xacro="http://ros.org/wiki/xacro">
-  <gazebo reference="table">
-    <minDepth>0.001</minDepth>
-    <material>Gazebo/SkyBlue</material>
-  </gazebo>
-  <gazebo>
-    <plugin filename="libgazebo_ros_control.so" name="gazebo_ros_control">
-      <robotNamespace>/ur5_sub</robotNamespace>
-    </plugin>
-  </gazebo>
-  <gazebo>
-    <plugin name="gazebo_ros_vacuum_gripper" filename="libgazebo_ros_vacuum_gripper.so">
-      <robotNamespace>/ur5_sub/vacuum_gripper</robotNamespace>
-      <bodyName>vacuum_gripper</bodyName>
-      <topicName>grasping</topicName>
-      <maxForce>50</maxForce>
-      <maxDistance>0.05</maxDistance>
-      <minDistance>0.01</minDistance>
-    </plugin>
-  </gazebo>
-  <gazebo reference="camera">
-    <sensor type="camera" name="camera">
-      <update_rate>30.0</update_rate>
-      <camera name="camera">
-        <horizontal_fov>${radians(100)}</horizontal_fov>
-        <image>
-          <width>800</width>
-          <height>800</height>
-          <format>R8G8B8</format>
-        </image>
-        <clip>
-          <near>0.02</near>
-          <far>300</far>
-        </clip>
-        <noise>
-          <type>gaussian</type>
-          <mean>0.0</mean>
-          <stddev>0.005</stddev>
-        </noise>
-      </camera>
-      <plugin name="camera_controller" filename="libgazebo_ros_camera.so">
-        <alwaysOn>true</alwaysOn>
-        <updateRate>0.0</updateRate>
-        <cameraName>camera</cameraName>
-        <imageTopicName>image_raw</imageTopicName>
-        <cameraInfoTopicName>camera_info</cameraInfoTopicName>
-        <frameName>camera</frameName>
-        <hackBaseline>0.0</hackBaseline>
-        <distortionK1>0.0</distortionK1>
-        <distortionK2>0.0</distortionK2>
-        <distortionK3>0.0</distortionK3>
-        <distortionT1>0.0</distortionT1>
-        <distortionT2>0.0</distortionT2>
+  <xacro:macro name = "ur5_gazebo">
+    <gazebo>
+      <plugin filename="libgazebo_ros_control.so" name="gazebo_ros_control">
+        <robotNamespace>/ur5_sub</robotNamespace>
       </plugin>
-    </sensor>
-  </gazebo>
+    </gazebo>
+    <gazebo>
+      <plugin name="gazebo_ros_vacuum_gripper" filename="libgazebo_ros_vacuum_gripper.so">
+        <robotNamespace>/ur5_sub/vacuum_gripper</robotNamespace>
+        <bodyName>vacuum_gripper</bodyName>
+        <topicName>grasping</topicName>
+        <maxForce>50</maxForce>
+        <maxDistance>0.07</maxDistance>
+        <minDistance>0.01</minDistance>
+      </plugin>
+    </gazebo>
+    <gazebo reference="camera">
+      <sensor type="camera" name="camera">
+        <update_rate>30.0</update_rate>
+        <camera name="camera">
+          <horizontal_fov>${radians(100)}</horizontal_fov>
+          <image>
+            <width>480</width>
+            <height>480</height>
+            <format>R8G8B8</format>
+          </image>
+          <clip>
+            <near>0.02</near>
+            <far>300</far>
+          </clip>
+          <noise>
+            <type>gaussian</type>
+            <mean>0.0</mean>
+            <stddev>0.005</stddev>
+          </noise>
+        </camera>
+        <plugin name="camera_controller" filename="libgazebo_ros_camera.so">
+          <alwaysOn>true</alwaysOn>
+          <updateRate>0.0</updateRate>
+          <cameraName>camera</cameraName>
+          <imageTopicName>image_raw</imageTopicName>
+          <cameraInfoTopicName>camera_info</cameraInfoTopicName>
+          <frameName>camera</frameName>
+          <hackBaseline>0.0</hackBaseline>
+          <distortionK1>0.0</distortionK1>
+          <distortionK2>0.0</distortionK2>
+          <distortionK3>0.0</distortionK3>
+          <distortionT1>0.0</distortionT1>
+          <distortionT2>0.0</distortionT2>
+        </plugin>
+      </sensor>
+    </gazebo>
+  </xacro:macro>
 </robot>

File: subbotinny_ur5_arm/urdf/ur5_pcb_table.urdf.xacro (robot description, xacro)
@@ -26,7 +26,8 @@
   <link name="camera" />
   <joint name="camera_joint" type="fixed">
-    <parent link="world" />
+    <parent link="base_link" />
     <child link="camera" />
-    <origin xyz="0 0.3 0.2" rpy="0 ${radians(-90)} 0" />
+    <origin xyz="0 0.7 0.01" rpy="0 ${radians(-90)} 0" />
   </joint>
+  <xacro:ur5_gazebo/>
 </robot>
