Commit message: Fixed models in world, added boxes and PCB to world

File: subbotinny_ur5_arm/urdf/ur5.urdf.xacro (robot description, xacro)
@@ -1,5 +1,5 @@
 <?xml version="1.0"?>
 <robot xmlns:xacro="http://www.ros.org/wiki/xacro">
-  <xacro:include filename="$(find subbotinny_ur5_vacuum)/urdf/ur.transmission.xacro" />
+  <xacro:include filename="$(find subbotinny_ur5_arm)/urdf/ur.transmission.xacro" />
   <!-- Inertia parameters -->
   <xacro:property name="base_mass" value="4.0" />  <!-- This mass might be incorrect -->

File: subbotinny_ur5_arm/urdf/ur5_pcb_table.urdf.xacro (robot description, xacro)
@@ -2,10 +2,6 @@
 <robot xmlns:xacro="http://ros.org/wiki/xacro"
        name="ur5" >
-  <!-- common stuff -->
-  <!-- <xacro:include filename="$(find ur5_vacuum)/urdf/common.gazebo.xacro" /> -->
-  <xacro:include filename="$(find subbotinny_ur5_vacuum)/urdf/ur5.material.xacro" />
-  <!-- ur5 -->
-  <xacro:include filename="$(find subbotinny_ur5_vacuum)/urdf/ur5.urdf.xacro" />
-  <xacro:include filename="$(find subbotinny_ur5_vacuum)/urdf/common.gazebo.xacro" />
+  <xacro:include filename="$(find subbotinny_ur5_arm)/urdf/ur5.urdf.xacro" />
+  <xacro:include filename="$(find subbotinny_ur5_arm)/urdf/common.gazebo.xacro" />
   <!-- arm -->
   <xacro:ur5_robot prefix="" joint_limited="true"
@@ -18,9 +14,8 @@
   />
   <link name="world" />
-  <!-- <xacro:rc0805 prefix="1" box_num="3"/> -->
   <joint name="world_joint" type="fixed">
     <parent link="world" />
     <child link = "base_link" />
-    <origin xyz="0 -0.4 0.105" rpy="0.0 0.0 0.0" />
+    <origin xyz="0 -0.3 0.105" rpy="0.0 0.0 0.0" />
   </joint>
   <link name="camera" />

Commit message: Added: urdf update

File: subbotinny_ur5_arm/urdf/ur5.urdf.xacro (robot description, xacro)
@@ -338,11 +338,4 @@
       <child link="${prefix}base"/>
     </joint>
-    <!-- Frame coincident with all-zeros TCP on UR controller -->
-    <link name="${prefix}tool0"/>
-    <joint name="${prefix}wrist_3_link-tool0_fixed_joint" type="fixed">
-      <origin xyz="0 ${wrist_3_length} 0" rpy="${pi/-2.0} 0 0"/>
-      <parent link="${prefix}wrist_3_link"/>
-      <child link="${prefix}tool0"/>
-    </joint>
   </xacro:macro>
 </robot>
