Commit message: Removed ns

File: ur5_vacuum_robot/urdf/common.gazebo.xacro (robot description, xacro)
@@ -4,5 +4,5 @@
     <gazebo>
       <plugin filename="libgazebo_ros_control.so" name="gazebo_ros_control">
-        <robotNamespace>/ur5_sub</robotNamespace>
+        <robotNamespace>/</robotNamespace>
       </plugin>
     </gazebo>

File: ur5_vacuum_robot/urdf/ur5_vacuum.urdf.xacro (robot description, xacro)
@@ -32,4 +32,10 @@
       </material>
     </visual>
+    <collision>
+      <origin rpy="0 0 0" xyz="0 0 0"/>
+      <geometry>
+      <cylinder radius="0.005" length="0.01"/>
+      </geometry>
+    </collision>
     <inertial>
       <origin rpy="0 0 0" xyz="0.000000 0.000000 0.000000"/>
