Commit message: Try to start vacuum

File: ur5_vacuum_robot/urdf/ur5_vacuum.urdf.xacro (robot description, xacro)
@@ -33,10 +33,4 @@
       </material>
     </visual>
-    <collision>
-      <origin rpy="0 0 0" xyz="0 0 0"/>
-      <geometry>
-      <cylinder radius="0.005" length="0.01"/>
-      </geometry>
-    </collision>
     <inertial>
       <origin rpy="0 0 0" xyz="0.000000 0.000000 0.000000"/>

Commit message: Try to fix vacuum 2

File: ur5_vacuum_robot/urdf/ur5_vacuum.urdf.xacro (robot description, xacro)
@@ -16,14 +16,14 @@
   <!-- vacuum gripper -->
   <joint name="gripper_joint" type="revolute">
-    <axis xyz="0 0 1" />
-    <parent link="tool0" />
+    <axis xyz="1 0 0" />
+    <parent link="ee_link" />
     <child link="vacuum_gripper" />
-    <origin rpy="0 0 0" xyz="0 0 0.01" />
-    <limit effort="50" velocity="50" lower="0" upper="0" />
+    <origin rpy="0 0 0" xyz="0 0 0" />
+    <limit effort="50" velocity="50" lower="-1" upper="1" />
   </joint>
   <link name="vacuum_gripper">
     <gravity>0</gravity>
     <visual>
-      <origin rpy="0 0 0" xyz="0 0 0"/>
+      <origin rpy="0 ${pi/2} 0" xyz="0 0 0"/>
       <geometry>
       <cylinder radius="0.005" length="0.01"/>

Commit message: Try to fix vacuum 3

File: ur5_vacuum_robot/urdf/ur5_vacuum.urdf.xacro (robot description, xacro)
@@ -16,16 +16,15 @@
   <!-- vacuum gripper -->
   <joint name="gripper_joint" type="revolute">
-    <axis xyz="1 0 0" />
+    <axis xyz="0 0 1" />
     <parent link="ee_link" />
     <child link="vacuum_gripper" />
-    <origin rpy="0 0 0" xyz="0 0 0" />
+    <origin rpy="0 ${pi/2} 0" xyz="0 0 0" />
     <limit effort="50" velocity="50" lower="-1" upper="1" />
   </joint>
   <link name="vacuum_gripper">
-    <gravity>0</gravity>
     <visual>
-      <origin rpy="0 ${pi/2} 0" xyz="0 0 0"/>
+      <origin rpy="0 0 0" xyz="0 0 0"/>
       <geometry>
-      <cylinder radius="0.005" length="0.01"/>
+        <cylinder radius="0.005" length="0.01"/>
       </geometry>
       <material name="red">
@@ -33,9 +32,13 @@
       </material>
     </visual>
-    <inertial>
-      <origin rpy="0 0 0" xyz="0.000000 0.000000 0.000000"/>
-      <mass value="0.0001"/>
-      <inertia ixx="1e-08" ixy="0" ixz="0" iyy="1e-08" iyz="0" izz="1e-08"/>
-    </inertial>
+    <collision>
+      <origin rpy="0 0 0" xyz="0 0 0"/>
+      <geometry>
+        <cylinder radius="0.005" length="0.01"/>
+      </geometry>
+    </collision>
+    <xacro:cylinder_inertial radius="0.005" length="0.01" mass="0.01">
+      <origin xyz="0.0 0.0 0.0" rpy="0 0 0" />
+    </xacro:cylinder_inertial>
   </link>
   <!-- camera -->

Commit message: Added: not final decision for vacuum (change to fixed joint)

File: ur5_vacuum_robot/urdf/ur5_vacuum.urdf.xacro (robot description, xacro)
@@ -15,5 +15,5 @@
   />
   <!-- vacuum gripper -->
-  <joint name="gripper_joint" type="revolute">
+  <joint name="gripper_joint" type="fixed">
     <axis xyz="0 0 1" />
     <parent link="ee_link" />

Commit message: Vacuum collision fix

File: ur5_vacuum_robot/urdf/ur5_vacuum.urdf.xacro (robot description, xacro)
@@ -24,7 +24,7 @@
   <link name="vacuum_gripper">
     <visual>
-      <origin rpy="0 0 0" xyz="0 0 0"/>
+      <origin rpy="0 0 0" xyz="0 0 0.005"/>
       <geometry>
-        <cylinder radius="0.005" length="0.01"/>
+        <cylinder radius="0.004" length="0.02"/>
       </geometry>
       <material name="red">
@@ -33,11 +33,11 @@
     </visual>
     <collision>
-      <origin rpy="0 0 0" xyz="0 0 0"/>
+      <origin rpy="0 0 0" xyz="0 0 0.005"/>
       <geometry>
-        <cylinder radius="0.005" length="0.01"/>
+        <cylinder radius="0.004" length="0.02"/>
       </geometry>
     </collision>
-    <xacro:cylinder_inertial radius="0.005" length="0.01" mass="0.01">
-      <origin xyz="0.0 0.0 0.0" rpy="0 0 0" />
+    <xacro:cylinder_inertial radius="0.004" length="0.02" mass="0.01">
+      <origin xyz="0.0 0.0 0.005" rpy="0 0 0" />
     </xacro:cylinder_inertial>
   </link>

Commit message: Vacuum collision fix 2

File: ur5_vacuum_robot/urdf/ur5_vacuum.urdf.xacro (robot description, xacro)
@@ -19,10 +19,10 @@
     <parent link="ee_link" />
     <child link="vacuum_gripper" />
-    <origin rpy="0 ${pi/2} 0" xyz="0 0 0" />
+    <origin rpy="0 ${pi/2} 0" xyz="0.005 0 0" />
     <limit effort="50" velocity="50" lower="-1" upper="1" />
   </joint>
   <link name="vacuum_gripper">
     <visual>
-      <origin rpy="0 0 0" xyz="0 0 0.005"/>
+      <origin rpy="0 0 0" xyz="0 0 0"/>
       <geometry>
         <cylinder radius="0.004" length="0.02"/>
@@ -33,5 +33,5 @@
     </visual>
     <collision>
-      <origin rpy="0 0 0" xyz="0 0 0.005"/>
+      <origin rpy="0 0 0" xyz="0 0 0"/>
       <geometry>
         <cylinder radius="0.004" length="0.02"/>
@@ -39,5 +39,5 @@
     </collision>
     <xacro:cylinder_inertial radius="0.004" length="0.02" mass="0.01">
-      <origin xyz="0.0 0.0 0.005" rpy="0 0 0" />
+      <origin xyz="0.0 0.0 0.0" rpy="0 0 0" />
     </xacro:cylinder_inertial>
   </link>

Commit message: Vacuum gripper fix

File: ur5_vacuum_robot/urdf/ur5_vacuum.urdf.xacro (robot description, xacro)
@@ -15,9 +15,9 @@
   />
   <!-- vacuum gripper -->
-  <joint name="gripper_joint" type="fixed">
+  <joint name="gripper_joint" type="revolute">
     <axis xyz="0 0 1" />
-    <parent link="ee_link" />
+    <parent link="wrist_3_link" />
     <child link="vacuum_gripper" />
-    <origin rpy="0 ${pi/2} 0" xyz="0.005 0 0" />
+    <origin rpy="${pi/2} 0 0" xyz="0 0.085 0" />
     <limit effort="50" velocity="50" lower="-1" upper="1" />
   </joint>
@@ -38,5 +38,5 @@
       </geometry>
     </collision>
-    <xacro:cylinder_inertial radius="0.004" length="0.02" mass="0.01">
+    <xacro:cylinder_inertial radius="0.004" length="0.02" mass="0.001">
       <origin xyz="0.0 0.0 0.0" rpy="0 0 0" />
     </xacro:cylinder_inertial>

Commit message: fix joint

File: ur5_vacuum_robot/urdf/ur5_vacuum.urdf.xacro (robot description, xacro)
@@ -55,5 +55,5 @@
   </link>
   <joint name="gripper_joint" type="revolute">
-    <axis xyz="0 0 0" />
+    <axis xyz="0 0 1" />
     <parent link="vacuum_gripper_base" />
     <child link="vacuum_gripper" />

Commit message: fix cameraa rotation

File: ur5_vacuum_robot/urdf/ur5_vacuum.urdf.xacro (robot description, xacro)
@@ -65,5 +65,5 @@
     <parent link="base_link" />
     <child link="camera" />
-    <origin xyz="0 0.6 0.01" rpy="0 ${-pi/2} 0" />
+    <origin xyz="0 0.6 0.01" rpy="0 ${-pi/2} ${-pi/2}" />
   </joint>
   <link name="camera" />

Commit message: Added conveyor

File: ur5_vacuum_robot/urdf/ur5_vacuum.urdf.xacro (robot description, xacro)
@@ -68,10 +68,10 @@
   </joint>
   <link name="camera" />
-  <xacro:include filename="$(find ur5_vacuum_robot)/urdf/ur5_gazebo.xacro" />
   <link name="world" />
-  <joint name="world_joint" type="fixed">
+  <joint name="world_joint_ur" type="fixed">
     <parent link="world" />
     <child link = "base_link" />
     <origin xyz="0 -0.3 0.105" rpy="0.0 0.0 0.0" />
   </joint>
+  <xacro:include filename="$(find ur5_vacuum_robot)/urdf/ur5_gazebo.xacro" />
 </robot>
