Commit message: Try to fix vacuum

File: ur5_vacuum_robot/urdf/ur5_gazebo.xacro (robot description, xacro)
@@ -1,5 +1,4 @@
 <?xml version="1.0"?>
 <robot xmlns:xacro="http://ros.org/wiki/xacro">
-  <xacro:macro name = "ur5_gazebo">
     <gazebo>
       <plugin name="gazebo_ros_vacuum_gripper" filename="libgazebo_ros_vacuum_gripper.so">
@@ -48,4 +47,3 @@
       </sensor>
     </gazebo>
-  </xacro:macro>
 </robot>

File: ur5_vacuum_robot/urdf/ur5_vacuum.urdf.xacro (robot description, xacro)
@@ -1,9 +1,7 @@
 <?xml version="1.0"?>
 <robot xmlns:xacro="http://ros.org/wiki/xacro"
-       name="ur5" >
+       name="ur5_vacuum" >
   <xacro:include filename="$(find ur_description)/urdf/common.gazebo.xacro" />
   <xacro:include filename="$(find ur_description)/urdf/ur5.urdf.xacro" />
-  <xacro:include filename="$(find ur5_vacuum_robot)/urdf/ur5_gazebo.xacro" />
-  <link name="world" />
   <!-- arm -->
   <xacro:ur5_robot prefix="" joint_limited="true"
@@ -16,10 +14,12 @@
     transmission_hw_interface = "hardware_interface/PositionJointInterface"
   />
-  <joint name="world_joint" type="fixed">
-    <parent link="world" />
-    <child link = "base_link" />
-    <origin xyz="0 -0.3 0.105" rpy="0.0 0.0 0.0" />
+  <!-- vacuum gripper -->
+  <joint name="gripper_joint" type="revolute">
+    <axis xyz="0 0 1" />
+    <parent link="tool0" />
+    <child link="vacuum_gripper" />
+    <origin rpy="0 0 0" xyz="0 0 0.01" />
+    <limit effort="50" velocity="50" lower="0" upper="0" />
   </joint>
-  <!-- vacuum gripper -->
   <link name="vacuum_gripper">
     <gravity>0</gravity>
@@ -29,6 +29,6 @@
       <cylinder radius="0.005" length="0.01"/>
       </geometry>
-      <material name="transparent">
-        <color rgba="0 0 0 0"/>
+      <material name="red">
+        <color rgba="0.8 0.0 0.0 1.0"/>
       </material>
     </visual>
@@ -39,19 +39,17 @@
     </inertial>
   </link>
-  <joint name="gripper_joint" type="fixed">
-    <axis xyz="1 0 0" />
-    <parent link="ee_link" />
-    <child link="vacuum_gripper" />
-    <origin rpy="0 1.5708 0" xyz="0.01 0 0" />
-<!--  <limit effort="50" velocity="50" lower="0" upper="0" />
-      <dynamics damping="0.0" friction="10"/> -->
-  </joint>
   <!-- camera -->
-  <link name="camera" />
   <joint name="camera_joint" type="fixed">
     <parent link="base_link" />
     <child link="camera" />
-    <origin xyz="0 0.7 0.01" rpy="0 ${radians(-90)} 0" />
+    <origin xyz="0 0.7 0.01" rpy="0 -1.5708 0" />
   </joint>
-  <xacro:ur5_gazebo/>
+  <link name="camera" />
+  <xacro:include filename="$(find ur5_vacuum_robot)/urdf/ur5_gazebo.xacro" />
+  <link name="world" />
+  <joint name="world_joint" type="fixed">
+    <parent link="world" />
+    <child link = "base_link" />
+    <origin xyz="0 -0.3 0.105" rpy="0.0 0.0 0.0" />
+  </joint>
 </robot>

Commit message: Vacuum gripper finally fixed

File: ur5_vacuum_robot/urdf/ur5_gazebo.xacro (robot description, xacro)
@@ -6,6 +6,6 @@
         <bodyName>vacuum_gripper</bodyName>
         <topicName>grasping</topicName>
-        <maxForce>50</maxForce>
-        <maxDistance>0.07</maxDistance>
+        <maxForce>10</maxForce>
+        <maxDistance>0.05</maxDistance>
         <minDistance>0.01</minDistance>
       </plugin>

File: ur5_vacuum_robot/urdf/ur5_vacuum.urdf.xacro (robot description, xacro)
@@ -15,10 +15,25 @@
   />
   <!-- vacuum gripper -->
-  <joint name="gripper_joint" type="revolute">
-    <axis xyz="0 0 1" />
+  <link name="vacuum_gripper_base">
+    <visual>
+      <origin rpy="0 0 0" xyz="0 0 0"/>
+      <geometry>
+        <cylinder radius="0.025" length="0.005"/>
+      </geometry>
+    </visual>
+    <collision>
+      <origin rpy="0 0 0" xyz="0 0 0"/>
+      <geometry>
+        <cylinder radius="0.025" length="0.005"/>
+      </geometry>
+    </collision>
+   <xacro:cylinder_inertial radius="0.025" length="0.005" mass="0.2">
+      <origin xyz="0.0 0.0 0.0" rpy="0 0 0" />
+    </xacro:cylinder_inertial>
+  </link>
+  <joint name="gripper_base_joint" type="fixed">
     <parent link="wrist_3_link" />
-    <child link="vacuum_gripper" />
-    <origin rpy="${pi/2} 0 0" xyz="0 0.085 0" />
-    <limit effort="50" velocity="50" lower="-1" upper="1" />
+    <child link="vacuum_gripper_base" />
+    <origin rpy="${-pi/2} 0 0" xyz="0 0.085 0" />
   </joint>
   <link name="vacuum_gripper">
@@ -26,20 +41,24 @@
       <origin rpy="0 0 0" xyz="0 0 0"/>
       <geometry>
-        <cylinder radius="0.004" length="0.02"/>
+        <cylinder radius="0.004" length="0.002"/>
       </geometry>
-      <material name="red">
-        <color rgba="0.8 0.0 0.0 1.0"/>
-      </material>
     </visual>
-    <collision>
+   <!-- <collision>
       <origin rpy="0 0 0" xyz="0 0 0"/>
       <geometry>
-        <cylinder radius="0.004" length="0.02"/>
+        <cylinder radius="0.004" length="0.002"/>
       </geometry>
-    </collision>
-    <xacro:cylinder_inertial radius="0.004" length="0.02" mass="0.001">
+    </collision> -->
+    <xacro:cylinder_inertial radius="0.004" length="0.002" mass="0.01">
       <origin xyz="0.0 0.0 0.0" rpy="0 0 0" />
     </xacro:cylinder_inertial>
   </link>
+  <joint name="gripper_joint" type="revolute">
+    <axis xyz="0 0 0" />
+    <parent link="vacuum_gripper_base" />
+    <child link="vacuum_gripper" />
+    <origin rpy="0 0 0" xyz="0 0 0.0035" />
+    <limit effort="20" velocity="1.0" lower="0" upper="0" />
+  </joint>
   <!-- camera -->
   <joint name="camera_joint" type="fixed">

Commit message: camera fix

File: ur5_vacuum_robot/urdf/ur5_gazebo.xacro (robot description, xacro)
@@ -22,5 +22,5 @@
           </image>
           <clip>
-            <near>0.02</near>
+            <near>0.005</near>
             <far>300</far>
           </clip>

File: ur5_vacuum_robot/urdf/ur5_vacuum.urdf.xacro (robot description, xacro)
@@ -65,5 +65,5 @@
     <parent link="base_link" />
     <child link="camera" />
-    <origin xyz="0 0.7 0.01" rpy="0 -1.5708 0" />
+    <origin xyz="0 0.6 0.01" rpy="0 ${-pi/2} 0" />
   </joint>
   <link name="camera" />

Commit message: Camera update

File: ur5_vacuum_robot/urdf/ur5_gazebo.xacro (robot description, xacro)
@@ -6,5 +6,5 @@
         <bodyName>vacuum_gripper</bodyName>
         <topicName>grasping</topicName>
-        <maxForce>1</maxForce>
+        <maxForce>0.001</maxForce>
         <maxDistance>0.05</maxDistance>
         <minDistance>0.01</minDistance>

File: ur5_vacuum_robot/urdf/ur5_vacuum.urdf.xacro (robot description, xacro)
@@ -41,5 +41,5 @@
       <origin rpy="0 0 0" xyz="0 0 0"/>
       <geometry>
-        <cylinder radius="0.004" length="0.002"/>
+        <cylinder radius="0.002" length="0.002"/>
       </geometry>
     </visual>
@@ -50,5 +50,5 @@
       </geometry>
     </collision> -->
-    <xacro:cylinder_inertial radius="0.004" length="0.002" mass="0.01">
+    <xacro:cylinder_inertial radius="0.002" length="0.002" mass="0.01">
       <origin xyz="0.0 0.0 0.0" rpy="0 0 0" />
     </xacro:cylinder_inertial>

Commit message: Added camera box

File: ur5_vacuum_robot/urdf/ur5_gazebo.xacro (robot description, xacro)
@@ -1,8 +1,8 @@
 <?xml version="1.0"?>
 <robot xmlns:xacro="http://ros.org/wiki/xacro">
-	<gazebo reference="vacuum_gripper_base">
+	<gazebo reference="gripper_camera">
 		<light name='test_light' type='directional'>
 			<intensity>1</intensity>
-			<pose>0 0.075 0.045 1.57 0 0</pose>
+			<pose>0 0.075 0.06 1.57 0 0</pose>
 			<!--attenuation>
 				<range>0.001</range>

File: ur5_vacuum_robot/urdf/ur5_vacuum.urdf.xacro (robot description, xacro)
@@ -68,4 +68,29 @@
   </joint>
   <link name="camera" />
+  <link name="gripper_camera">
+  	<collision>
+  		<origin xyz="0 0 0" rpy="0 0 0"/>
+  		<geometry>
+  			<box size="0.02 0.02 0.02"/>
+  		</geometry>
+  	</collision>
+  	<visual>
+  		<origin xyz="0 0 0" rpy="0 0 0"/>
+  		<geometry>
+  			<box size="0.02 0.02 0.02"/>
+  		</geometry>
+  	</visual>
+  	<inertial>
+  		<mass value="1e-5"/>
+  		<origin xyz="0 0 0" rpy="0 0 0"/>
+  		<inertia ixx="1e-6" ixy="0" ixz="0" iyy="1e-6" iyz="0" izz="1e-6"/>
+  	</inertial>
+  </link>
+  <joint name="gripper_camera_joint" type="fixed">
+  	<axis xyz="0 1 0"/>
+  	<origin xyz="-0.02 0.0 0.055" rpy="0 0 0"/>
+  	<parent link="ee_link"/>
+  	<child link="gripper_camera"/>
+  </joint>
   <link name="world" />
   <joint name="world_joint_ur" type="fixed">

Commit message: Added second camera

File: ur5_vacuum_robot/urdf/ur5_gazebo.xacro (robot description, xacro)
@@ -1,13 +1,49 @@
 <?xml version="1.0"?>
 <robot xmlns:xacro="http://ros.org/wiki/xacro">
+  <gazebo reference="gripper_camera">
+    <mu1>0.2</mu1>
+    <mu2>0.2</mu2>
+    <material>Gazebo/Green</material>
+  </gazebo>
+  <gazebo reference="gripper_camera">
+    <sensor type="camera" name="gripper_camera">
+      <update_rate>30.0</update_rate>
+      <camera name="head">
+        <horizontal_fov>${radians(100)}</horizontal_fov>
+        <image>
+          <width>800</width>
+          <height>800</height>
+          <format>R8G8B8</format>
+        </image>
+        <clip>
+          <near>0.02</near>
+          <far>300</far>
+        </clip>
+        <noise>
+          <type>gaussian</type>
+          <mean>0.0</mean>
+          <stddev>0.007</stddev>
+        </noise>
+      </camera>
+      <plugin name="camera_controller" filename="libgazebo_ros_camera.so">
+        <alwaysOn>true</alwaysOn>
+        <updateRate>0.0</updateRate>
+        <cameraName>gripper_camera</cameraName>
+        <imageTopicName>image_raw</imageTopicName>
+        <cameraInfoTopicName>camera_info</cameraInfoTopicName>
+        <frameName>camera</frameName>
+        <hackBaseline>0.0</hackBaseline>
+        <distortionK1>0.0</distortionK1>
+        <distortionK2>0.0</distortionK2>
+        <distortionK3>0.0</distortionK3>
+        <distortionT1>0.0</distortionT1>
+        <distortionT2>0.0</distortionT2>
+      </plugin>
+    </sensor>
+  </gazebo>
 	<gazebo reference="gripper_camera">
 		<light name='test_light' type='directional'>
 			<intensity>1</intensity>
 			<pose>0 0.075 0.06 1.57 0 0</pose>
-			<!--attenuation>
-				<range>0.001</range>
-				<linear>0.2</linear>
-				<constant>0.8</constant>
-			</attenuation-->
 		</light>
 		<plugin name='light_control' filename='libFlashLightPlugin.so'>
@@ -31,39 +67,39 @@
 		</plugin>
 	</gazebo>
-    <gazebo reference="camera">
-      <sensor type="camera" name="camera">
-        <update_rate>30.0</update_rate>
-        <camera name="camera">
-          <horizontal_fov>${radians(100)}</horizontal_fov>
-          <image>
-            <width>480</width>
-            <height>480</height>
-            <format>R8G8B8</format>
-          </image>
-          <clip>
-            <near>0.005</near>
-            <far>300</far>
-          </clip>
-          <noise>
-            <type>gaussian</type>
-            <mean>0.0</mean>
-            <stddev>0.005</stddev>
-          </noise>
-        </camera>
-        <plugin name="camera_controller" filename="libgazebo_ros_camera.so">
-          <alwaysOn>true</alwaysOn>
-          <updateRate>0.0</updateRate>
-          <cameraName>camera</cameraName>
-          <imageTopicName>image_raw</imageTopicName>
-          <cameraInfoTopicName>camera_info</cameraInfoTopicName>
-          <frameName>camera</frameName>
-          <hackBaseline>0.0</hackBaseline>
-          <distortionK1>0.0</distortionK1>
-          <distortionK2>0.0</distortionK2>
-          <distortionK3>0.0</distortionK3>
-          <distortionT1>0.0</distortionT1>
-          <distortionT2>0.0</distortionT2>
-        </plugin>
-      </sensor>
-    </gazebo>
+  <gazebo reference="camera">
+    <sensor type="camera" name="camera">
+      <update_rate>30.0</update_rate>
+      <camera name="camera">
+        <horizontal_fov>${radians(100)}</horizontal_fov>
+        <image>
+          <width>480</width>
+          <height>480</height>
+          <format>R8G8B8</format>
+        </image>
+        <clip>
+          <near>0.005</near>
+          <far>300</far>
+        </clip>
+        <noise>
+          <type>gaussian</type>
+          <mean>0.0</mean>
+          <stddev>0.005</stddev>
+        </noise>
+      </camera>
+      <plugin name="camera_controller" filename="libgazebo_ros_camera.so">
+        <alwaysOn>true</alwaysOn>
+        <updateRate>0.0</updateRate>
+        <cameraName>camera</cameraName>
+        <imageTopicName>image_raw</imageTopicName>
+        <cameraInfoTopicName>camera_info</cameraInfoTopicName>
+        <frameName>camera</frameName>
+        <hackBaseline>0.0</hackBaseline>
+        <distortionK1>0.0</distortionK1>
+        <distortionK2>0.0</distortionK2>
+        <distortionK3>0.0</distortionK3>
+        <distortionT1>0.0</distortionT1>
+        <distortionT2>0.0</distortionT2>
+      </plugin>
+    </sensor>
+  </gazebo>
 </robot>
