Commit message: Updated cobnveyor params

File: ur5_vacuum_demo/urdf/pcb.urdf (robot description, URDF)
Before this commit: robot pcb, 1 links, 0 joints
Links:
- link pcb: mass 0.00001 -> 0.1

File: ur5_vacuum_robot/urdf/ur5_gazebo.xacro (robot description, xacro)
@@ -6,7 +6,7 @@
         <bodyName>vacuum_gripper</bodyName>
         <topicName>grasping</topicName>
-        <maxForce>0.001</maxForce>
-        <maxDistance>0.05</maxDistance>
-        <minDistance>0.01</minDistance>
+        <maxForce>0.00000001</maxForce>
+        <maxDistance>0.001</maxDistance>
+        <minDistance>0.00001</minDistance>
       </plugin>
     </gazebo>

Commit message: Update parameters

File: ur5_vacuum_demo/urdf/pcb.urdf (robot description, URDF)
Before this commit: robot pcb, 1 links, 0 joints
Links:
- link pcb: mass 0.1 -> 1

File: ur5_vacuum_robot/urdf/ur5_gazebo.xacro (robot description, xacro)
@@ -6,5 +6,5 @@
         <bodyName>vacuum_gripper</bodyName>
         <topicName>grasping</topicName>
-        <maxForce>0.00000001</maxForce>
+        <maxForce>0.000000000001</maxForce>
         <maxDistance>0.001</maxDistance>
         <minDistance>0.00001</minDistance>

Commit message: Fixed pcb model, upd algo

File: ur5_vacuum_demo/urdf/pcb.urdf (robot description, URDF)
Before this commit: robot pcb, 1 links, 0 joints
Links:
- link pcb: mass 1 -> 2; geometry collision box size=0.08 0.12 0.002; visual mesh filename=package://ur5_vacuum_demo/urdf/models/board.stl scale=0.001 0.001 0.001

Commit message: Added: .dae model

File: ur5_vacuum_demo/urdf/pcb.urdf (robot description, URDF)
Before this commit: robot pcb, 1 links, 0 joints
Links:
- link pcb: geometry collision mesh filename=package://ur5_vacuum_demo/urdf/models/textured_panel.dae scale=0.001 0.001 0.001; visual mesh filename=package://ur5_vacuum_demo/urdf/models/textured_panel.dae scale=0.001 0.001 0.001

Commit message: Fixed pcb size

File: ur5_vacuum_demo/urdf/pcb.urdf (robot description, URDF)
Before this commit: robot pcb, 1 links, 0 joints
Links:
- link pcb: geometry collision mesh filename=package://ur5_vacuum_demo/urdf/models/textured_panel.dae scale=0.3 0.3 0.3; visual mesh filename=package://ur5_vacuum_demo/urdf/models/textured_panel.dae scale=0.3 0.3 0.3
