Commit message: dev

File: ur5_vacuum_demo/urdf/component_0402.urdf (robot description, URDF)
Before this commit: robot box_g, 1 links, 0 joints
Links:
- link box_g: geometry collision box size=0.02 0.01 0.005; visual box size=0.02 0.01 0.005

File: ur5_vacuum_robot/urdf/ur5_gazebo.xacro (robot description, xacro)
@@ -6,5 +6,5 @@
         <bodyName>vacuum_gripper</bodyName>
         <topicName>grasping</topicName>
-        <maxForce>10</maxForce>
+        <maxForce>1</maxForce>
         <maxDistance>0.05</maxDistance>
         <minDistance>0.01</minDistance>

Commit message: dev

File: ur5_vacuum_demo/urdf/component_0402.urdf (robot description, URDF)
Before this commit: robot box_g, 1 links, 0 joints
Links:
- link box_g: geometry collision box size=0.01 0.005 0.0025; visual box size=0.01 0.005 0.0025

Commit message: Added realism

File: ur5_vacuum_demo/urdf/component_0402.urdf (robot description, URDF)
Before this commit: robot box_g, 1 links, 0 joints
Links:
- link box_g: mass 0.00875 -> 0.1; geometry collision box size=0.002 0.00125 0.0008; visual box size=0.002 0.00125 0.0008

File: ur5_vacuum_demo/urdf/pcb.urdf (robot description, URDF)
Before this commit: robot pcb, 1 links, 0 joints
Links:
- link pcb: mass 2 -> 10

File: ur5_vacuum_robot/urdf/ur5_gazebo.xacro (robot description, xacro)
@@ -6,5 +6,5 @@
         <bodyName>vacuum_gripper</bodyName>
         <topicName>grasping</topicName>
-        <maxForce>0.000000000001</maxForce>
+        <maxForce>0.0001</maxForce>
         <maxDistance>0.001</maxDistance>
         <minDistance>0.00001</minDistance>

File: ur5_vacuum_robot/urdf/ur5_vacuum.urdf.xacro (robot description, xacro)
@@ -41,5 +41,5 @@
       <origin rpy="0 0 0" xyz="0 0 0"/>
       <geometry>
-        <cylinder radius="0.002" length="0.002"/>
+        <cylinder radius="0.001" length="0.0005"/>
       </geometry>
     </visual>
@@ -50,14 +50,14 @@
       </geometry>
     </collision> -->
-    <xacro:cylinder_inertial radius="0.002" length="0.002" mass="0.01">
+    <xacro:cylinder_inertial radius="0.001" length="0.0005" mass="0.0001">
       <origin xyz="0.0 0.0 0.0" rpy="0 0 0" />
     </xacro:cylinder_inertial>
   </link>
   <joint name="gripper_joint" type="revolute">
-    <axis xyz="0 0 1" />
+    <axis xyz="0 0 0" />
     <parent link="vacuum_gripper_base" />
     <child link="vacuum_gripper" />
-    <origin rpy="0 0 0" xyz="0 0 0.0035" />
-    <limit effort="20" velocity="1.0" lower="0" upper="0" />
+    <origin rpy="0 0 0" xyz="0 0 0.00275" />
+    <limit effort="0.0001" velocity="0.001" lower="0" upper="0" />
   </joint>
   <!-- camera -->
