Commit message: Try to make conveyor controller

File: ur5_vacuum_conveyor/urdf/ur5_vacuum_conveyor.urdf.xacro (robot description, xacro)
@@ -24,15 +24,24 @@
 </link>
 <gazebo reference="conveyor_base">
-  <mu1>0</mu1>
-  <mu2>0</mu2>
+  <mu1>1</mu1>
+  <mu2>1</mu2>
   <material>Gazebo/FlatBlack</material>
 </gazebo>
 <link name="world" />
-  <joint name="conveyor_joint" type="prismatic">
-    <parent link="world" />
-    <child link = "conveyor_base" />
-    <origin xyz="0 0 0.05" rpy="0.0 0.0 0.0" />
-    <axis xyz="0 1 0"/>
-    <limit upper = "0" lower="-4" effort="1000" velocity="0.2"/>
+<joint name="conveyor_joint" type="prismatic">
+  <parent link="world" />
+  <child link = "conveyor_base" />
+  <origin xyz="0 0 0.05" rpy="0.0 0.0 0.0" />
+  <axis xyz="0 1 0"/>
+  <limit upper = "0" lower="-4" effort="1" velocity="1"/>
+</joint>
+<transmission name="conveyor_joint_trans">
+  <type>transmission_interface/SimpleTransmission</type>
+  <joint name="conveyor_joint">
+    <hardwareInterface>hardware_interface/EffortJointInterface</hardwareInterface>
   </joint>
+  <actuator name="conveyor_motor">
+    <mechanicalReduction>1</mechanicalReduction>
+  </actuator>
+</transmission>
 </robot>

Commit message: Conveyor algo update

File: ur5_vacuum_conveyor/urdf/ur5_vacuum_conveyor.urdf.xacro (robot description, xacro)
@@ -36,12 +36,3 @@
   <limit upper = "0" lower="-4" effort="1" velocity="1"/>
 </joint>
-<transmission name="conveyor_joint_trans">
-  <type>transmission_interface/SimpleTransmission</type>
-  <joint name="conveyor_joint">
-    <hardwareInterface>hardware_interface/EffortJointInterface</hardwareInterface>
-  </joint>
-  <actuator name="conveyor_motor">
-    <mechanicalReduction>1</mechanicalReduction>
-  </actuator>
-</transmission>
 </robot>

Commit message: Added: spawn pcb to conveyor

File: ur5_vacuum_conveyor/urdf/ur5_vacuum_conveyor.urdf.xacro (robot description, xacro)
@@ -6,5 +6,5 @@
     <origin xyz="0 0 0" rpy="0 0 0"/>
     <geometry>
-      <box size="0.3 5 0.1"/>
+      <box size="0.3 2 0.1"/>
     </geometry>
   </visual>
@@ -12,5 +12,5 @@
     <origin xyz="0 0 0" rpy="0 0 0"/>
     <geometry>
-      <box size="0.3 5 0.1"/>
+      <box size="0.3 2 0.1"/>
     </geometry>
   </collision>
@@ -29,10 +29,8 @@
 </gazebo>
 <link name="world" />
-<joint name="conveyor_joint" type="prismatic">
+<joint name="conveyor_joint" type="fixed">
   <parent link="world" />
   <child link = "conveyor_base" />
   <origin xyz="0 0 0.05" rpy="0.0 0.0 0.0" />
-  <axis xyz="0 1 0"/>
-  <limit upper = "0" lower="-4" effort="1" velocity="1"/>
 </joint>
 </robot>

Commit message: Updated sizes

File: ur5_vacuum_conveyor/urdf/ur5_vacuum_conveyor.urdf.xacro (robot description, xacro)
@@ -6,5 +6,5 @@
     <origin xyz="0 0 0" rpy="0 0 0"/>
     <geometry>
-      <box size="0.3 2 0.1"/>
+      <box size="0.5 2 0.1"/>
     </geometry>
   </visual>
@@ -12,5 +12,5 @@
     <origin xyz="0 0 0" rpy="0 0 0"/>
     <geometry>
-      <box size="0.3 2 0.1"/>
+      <box size="0.5 2 0.1"/>
     </geometry>
   </collision>

File: ur5_vacuum_demo/urdf/component_0402.urdf (robot description, URDF)
Before this commit: robot box_g, 1 links, 0 joints
Links:
- link box_g: geometry collision box size=0.0008 0.002 0.001; visual box size=0.0008 0.002 0.001

File: ur5_vacuum_demo/urdf/pcb.urdf (robot description, URDF)
Before this commit: robot pcb, 1 links, 0 joints
Links:
- link pcb: geometry collision mesh filename=package://ur5_vacuum_demo/urdf/models/textured_panel.dae scale=0.5 0.5 0.5; visual mesh filename=package://ur5_vacuum_demo/urdf/models/textured_panel.dae scale=0.5 0.5 0.5
